Commit message: Update objectives and remove manual_grasp_link

File: src/kinova_gen3_base_config/description/gripper_and_camera.xacro (robot description, xacro)
@@ -8,11 +8,11 @@
   <xacro:include filename="$(find picknik_accessories)/descriptions/sensors/realsense_d415.urdf.xacro"/>
   <!-- Create parent link -->
-  <!-- Moveit Studio requires a link name called manual_grasp_link to perform quick tasks such as inspect surface -->
-  <link name="manual_grasp_link" />
+  <!-- We use a link name called grasp_link to perform built-in Objectives such as inspect surface without modification. -->
+  <link name="grasp_link" />
   <!-- Create bracelet link -->
   <link name="bracelet_link" />
   <joint name="bracelet_joint" type="fixed">
-    <origin xyz="0 -0.031521 -0.1787672" rpy="${pi / 180.0 * 170} 0 0" />
-    <parent link="manual_grasp_link" />
+    <origin xyz="0 -0.031521 -0.1787672" rpy="0 0 0" />
+    <parent link="grasp_link" />
     <child link="bracelet_link" />
   </joint>

File: src/kinova_gen3_base_config/description/picknik_kinova_gen3.xacro (robot description, xacro)
@@ -121,11 +121,10 @@
       <origin xyz="0 0 0.16" rpy="0 0 0"/>
     </joint>
-    <!-- Moveit Studio requires a link name called manual_grasp_link to perform quick tasks such as inspect surface -->
-    <!-- we add this link here and make it coincident with the manual_grasp_link but rotate it to put the camera normal to the surface -->
-    <link name="manual_grasp_link"/>
-    <joint name="manual_grasp_joint" type="fixed">
+    <!-- This link aligns the axes of the grasp frame to our required convention for motion planning tasks. -->
+    <link name="grasp_link"/>
+    <joint name="grasp_link_joint" type="fixed">
       <parent link="$(arg prefix)end_effector_link"/>
-      <child link = "manual_grasp_link"/>
-      <origin xyz="0 0 0.15" rpy="${3.14 / 180.0 * 10} 0 0"/>
+      <child link = "grasp_link"/>
+      <origin xyz="0 0 0.15" rpy="0 0 0"/>
     </joint>
     <!-- Camera External -->
