Commit message: Set initial joint positions during render
Pass the default values in the `config/initial_positions.yaml` file to
the initial_positions parameter of the load_robot macro during render of
the kinova to set it to the home position by default.

Point to updated ros2_kortex submodule commit that enables the
initial_positions parameter in the load_robot macro.

Point to latest ros2_robotiq_gripper submodule commit.

File: src/kinova_gen3_base_config/description/picknik_kinova_gen3.xacro (robot description, xacro)
@@ -32,4 +32,8 @@
     <!-- World is centered under base_link of the robot, on the ground -->
     <link name="world"/>
+    <!-- initial position for simulations (Mock Hardware, Gazebo, Ignition) -->
+    <xacro:arg name="initial_positions_file" default="$(find kinova_gen3_base_config)/config/initial_positions.yaml"/>
+    <!-- convert to property to use substitution in function -->
+    <xacro:property name="initial_positions_file" default="$(arg initial_positions_file)"/>
     <!-- Load the robot -->
     <xacro:load_robot
@@ -56,5 +60,6 @@
       use_external_cable="$(arg use_external_cable)"
       gripper_max_velocity="$(arg gripper_joint_name)"
-      gripper_max_force="$(arg gripper_max_force)" >
+      gripper_max_force="$(arg gripper_max_force)"
+      initial_positions="${xacro.load_yaml(initial_positions_file)}" >
       <origin xyz="0 0 0.0" rpy="0 0 0" />
     </xacro:load_robot>

File: src/picknik_kinova_gen3_site_config/description/picknik_kinova_gen3.xacro (robot description, xacro)
@@ -32,4 +32,8 @@
     <!-- World is centered under base_link of the robot, on the ground -->
     <link name="world"/>
+    <!-- initial position for simulations (Mock Hardware, Gazebo, Ignition) -->
+    <xacro:arg name="initial_positions_file" default="$(find picknik_kinova_gen3_site_config)/config/initial_positions.yaml"/>
+    <!-- convert to property to use substitution in function -->
+    <xacro:property name="initial_positions_file" default="$(arg initial_positions_file)"/>
     <!-- Load the robot -->
     <xacro:load_robot
@@ -56,5 +60,6 @@
       use_external_cable="$(arg use_external_cable)"
       gripper_max_velocity="$(arg gripper_joint_name)"
-      gripper_max_force="$(arg gripper_max_force)" >
+      gripper_max_force="$(arg gripper_max_force)"
+      initial_positions="${xacro.load_yaml(initial_positions_file)}" >
       <origin xyz="0 0 0.0" rpy="0 0 0" />
     </xacro:load_robot>

Commit message: fix grasp_link in mock config

File: src/kinova_gen3_base_config/description/picknik_kinova_gen3.xacro (robot description, xacro)
@@ -124,5 +124,5 @@
     <link name="grasp_link"/>
     <joint name="grasp_link_joint" type="fixed">
-      <parent link="$(arg prefix)end_effector_link"/>
+      <parent link="robotiq_85_base_link"/>
       <child link = "grasp_link"/>
       <origin xyz="0 0 0.15" rpy="0 0 0"/>
