Commit message: fix URDF
Signed-off-by: Paul Gesel <paulgesel@gmail.com>

File: src/kinova_gen3_mujoco_config/description/picknik_kinova_gen3.xacro (robot description, xacro)
@@ -482,5 +482,5 @@
       <parent link="robotiq_85_base_link"/>
       <child link="robotiq_85_right_knuckle_link"/>
-      <axis xyz="0 -1 0"/>
+      <axis xyz="0 1 0"/>
       <origin rpy="0 0 0" xyz="-0.03060114 0.0 0.05490452"/>
       <limit effort="50" lower="-0.8" upper="0.0" velocity="0.5"/>
@@ -507,5 +507,5 @@
       <parent link="robotiq_85_base_link"/>
       <child link="robotiq_85_right_inner_knuckle_link"/>
-      <axis xyz="0 -1 0"/>
+      <axis xyz="0 1 0"/>
       <origin rpy="0 0 0" xyz="-0.0127 0.0 0.06142"/>
       <mimic joint="robotiq_85_left_knuckle_joint" multiplier="-1"/>
@@ -521,5 +521,5 @@
       <parent link="robotiq_85_right_finger_link"/>
       <child link="robotiq_85_right_finger_tip_link"/>
-      <axis xyz="0 -1 0"/>
+      <axis xyz="0 1 0"/>
       <origin rpy="0 0 0" xyz="-0.00563134 0.0 0.04718515"/>
       <mimic joint="robotiq_85_left_knuckle_joint"/>

Commit message: Remove mimic joint details
They are not used in the ros2_control mujoco SystemInterface

File: src/kinova_gen3_mujoco_config/description/picknik_kinova_gen3.xacro (robot description, xacro)
@@ -478,5 +478,5 @@
       <origin rpy="0 0 0" xyz="-0.03060114 0.0 0.05490452"/>
       <limit effort="50" lower="-0.8" upper="0.0" velocity="0.5"/>
-      <mimic joint="robotiq_85_left_knuckle_joint" multiplier="-1"/>
+      <!-- <mimic joint="robotiq_85_left_knuckle_joint" multiplier="-1"/> -->
     </joint>
     <joint name="robotiq_85_left_finger_joint" type="fixed">
@@ -495,5 +495,5 @@
       <axis xyz="0 -1 0"/>
       <origin rpy="0 0 0" xyz="0.0127 0.0 0.06142"/>
-      <mimic joint="robotiq_85_left_knuckle_joint"/>
+      <!-- <mimic joint="robotiq_85_left_knuckle_joint"/> -->
     </joint>
     <joint name="robotiq_85_right_inner_knuckle_joint" type="continuous">
@@ -502,5 +502,5 @@
       <axis xyz="0 1 0"/>
       <origin rpy="0 0 0" xyz="-0.0127 0.0 0.06142"/>
-      <mimic joint="robotiq_85_left_knuckle_joint" multiplier="-1"/>
+      <!-- <mimic joint="robotiq_85_left_knuckle_joint" multiplier="1"/> -->
     </joint>
     <joint name="robotiq_85_left_finger_tip_joint" type="continuous">
@@ -509,5 +509,5 @@
       <axis xyz="0 -1 0"/>
       <origin rpy="0 0 0" xyz="0.00563134 0.0 0.04718515"/>
-      <mimic joint="robotiq_85_left_knuckle_joint" multiplier="-1"/>
+      <!-- <mimic joint="robotiq_85_left_knuckle_joint" multiplier="-1"/> -->
     </joint>
     <joint name="robotiq_85_right_finger_tip_joint" type="continuous">
@@ -516,5 +516,5 @@
       <axis xyz="0 1 0"/>
       <origin rpy="0 0 0" xyz="-0.00563134 0.0 0.04718515"/>
-      <mimic joint="robotiq_85_left_knuckle_joint"/>
+      <!-- <mimic joint="robotiq_85_left_knuckle_joint" multiplier="-1"/> -->
     </joint>
     <!-- Environment -->
@@ -682,30 +682,20 @@
       </joint>
       <joint name="robotiq_85_right_knuckle_joint">
-        <param name="mimic">robotiq_85_left_knuckle_joint</param>
-        <param name="multiplier">-1</param>
         <state_interface name="position"/>
         <state_interface name="velocity"/>
       </joint>
       <joint name="robotiq_85_left_inner_knuckle_joint">
-        <param name="mimic">robotiq_85_left_knuckle_joint</param>
-        <param name="multiplier">1</param>
         <state_interface name="position"/>
         <state_interface name="velocity"/>
       </joint>
       <joint name="robotiq_85_right_inner_knuckle_joint">
-        <param name="mimic">robotiq_85_left_knuckle_joint</param>
-        <param name="multiplier">-1</param>
         <state_interface name="position"/>
         <state_interface name="velocity"/>
       </joint>
       <joint name="robotiq_85_left_finger_tip_joint">
-        <param name="mimic">robotiq_85_left_knuckle_joint</param>
-        <param name="multiplier">-1</param>
         <state_interface name="position"/>
         <state_interface name="velocity"/>
       </joint>
       <joint name="robotiq_85_right_finger_tip_joint">
-        <param name="mimic">robotiq_85_left_knuckle_joint</param>
-        <param name="multiplier">1</param>
         <state_interface name="position"/>
         <state_interface name="velocity"/>

Commit message: Correct limits for knuckle joint and add mimic joints back

File: src/kinova_gen3_mujoco_config/description/picknik_kinova_gen3.xacro (robot description, xacro)
@@ -477,6 +477,6 @@
       <axis xyz="0 1 0"/>
       <origin rpy="0 0 0" xyz="-0.03060114 0.0 0.05490452"/>
-      <limit effort="50" lower="-0.8" upper="0.0" velocity="0.5"/>
-      <!-- <mimic joint="robotiq_85_left_knuckle_joint" multiplier="-1"/> -->
+      <limit effort="50" lower="0.0" upper="0.8" velocity="0.5"/>
+      <mimic joint="robotiq_85_left_knuckle_joint" multiplier="1"/>
     </joint>
     <joint name="robotiq_85_left_finger_joint" type="fixed">
@@ -495,5 +495,5 @@
       <axis xyz="0 -1 0"/>
       <origin rpy="0 0 0" xyz="0.0127 0.0 0.06142"/>
-      <!-- <mimic joint="robotiq_85_left_knuckle_joint"/> -->
+      <mimic joint="robotiq_85_left_knuckle_joint" multiplier="1"/>
     </joint>
     <joint name="robotiq_85_right_inner_knuckle_joint" type="continuous">
@@ -502,5 +502,5 @@
       <axis xyz="0 1 0"/>
       <origin rpy="0 0 0" xyz="-0.0127 0.0 0.06142"/>
-      <!-- <mimic joint="robotiq_85_left_knuckle_joint" multiplier="1"/> -->
+      <mimic joint="robotiq_85_left_knuckle_joint" multiplier="1"/>
     </joint>
     <joint name="robotiq_85_left_finger_tip_joint" type="continuous">
@@ -509,5 +509,5 @@
       <axis xyz="0 -1 0"/>
       <origin rpy="0 0 0" xyz="0.00563134 0.0 0.04718515"/>
-      <!-- <mimic joint="robotiq_85_left_knuckle_joint" multiplier="-1"/> -->
+      <mimic joint="robotiq_85_left_knuckle_joint" multiplier="-1"/>
     </joint>
     <joint name="robotiq_85_right_finger_tip_joint" type="continuous">
@@ -516,5 +516,5 @@
       <axis xyz="0 1 0"/>
       <origin rpy="0 0 0" xyz="-0.00563134 0.0 0.04718515"/>
-      <!-- <mimic joint="robotiq_85_left_knuckle_joint" multiplier="-1"/> -->
+      <mimic joint="robotiq_85_left_knuckle_joint" multiplier="-1"/>
     </joint>
     <!-- Environment -->

Commit message: fix MJCF world position and add take_snapshot
Signed-off-by: Paul Gesel <paulgesel@gmail.com>

File: src/kinova_gen3_mujoco_config/description/picknik_kinova_gen3.xacro (robot description, xacro)
@@ -243,14 +243,14 @@
         <origin rpy="0 0 0" xyz="0 0 0"/>
         <geometry>
-          <mesh filename="package://kortex_description/arms/gen3/7dof/meshes/bracelet_no_vision_link.dae"/>
-        </geometry>
-        <material name="">
-          <color rgba="0.75294 0.75294 0.75294 1"/>
-        </material>
-      </visual>
-      <collision>
-        <origin rpy="0 0 0" xyz="0 0 0"/>
-        <geometry>
-          <mesh filename="package://kortex_description/arms/gen3/7dof/meshes/bracelet_no_vision_link.dae"/>
+          <mesh filename="package://kortex_description/arms/gen3/7dof/meshes/bracelet_with_vision_link.dae"/>
+        </geometry>
+        <material name="">
+          <color rgba="0.75294 0.75294 0.75294 1"/>
+        </material>
+      </visual>
+      <collision>
+        <origin rpy="0 0 0" xyz="0 0 0"/>
+        <geometry>
+          <mesh filename="package://kortex_description/arms/gen3/7dof/meshes/bracelet_with_vision_link.dae"/>
         </geometry>
       </collision>
@@ -522,60 +522,20 @@
       <origin xyz="0 0 -0.145" rpy="0 0 0"/>
     </xacro:cube>
-    <!-- wrist realsense -->
-    <!-- <xacro:if value="$(arg wrist_realsense)"> -->
-    <!--   <link name="wrist_camera_link"/> -->
-    <!---->
-    <!--   <joint name="wrist_camera_joint" type="fixed"> -->
-    <!--     <parent link="$(arg prefix)bracelet_link"/> -->
-    <!--     <child link = "wrist_camera_link"/> -->
-    <!--     <origin xyz="0 -0.06841 -0.05044" rpy="0 ${3.14 / 180.0 * 100} -1.5708"/> -->
-    <!--   </joint> -->
-    <!---->
-    <!--   <xacro:realsense_d415 parent="wrist_camera_link" name="wrist_mounted_camera"> -->
-    <!--     <origin xyz="0 0 0" rpy="0 0 0"/> -->
-    <!--   </xacro:realsense_d415> -->
-      <!-- Bracket -->
-    <!--   <link name="wrist_camera_link_visual"> -->
-    <!--     <inertial> -->
-    <!--       <origin xyz="0.000281 0.011402 -0.029798" rpy="0 0 0" /> -->
-    <!--       <mass value="0.5" /> -->
-    <!--       <inertia ixx="0.000587" ixy="3E-06" ixz="3E-06" iyy="0.000369" iyz="-0.000118" izz="0.000609" /> -->
-    <!--     </inertial> -->
-    <!--     <visual> -->
-    <!--       <origin xyz="0 0 0" rpy="0 0 0" /> -->
-    <!--       <geometry> -->
-    <!--         <mesh filename="package://picknik_accessories/descriptions/brackets/kinova_realsense_camera_adapter/realsense_bracket_for_kinova.dae" /> -->
-    <!--       </geometry> -->
-    <!--     </visual> -->
-    <!--     <collision> -->
-    <!--       <origin xyz="0 0 0" rpy="0 0 0" /> -->
-    <!--       <geometry> -->
-    <!--         <mesh filename="package://picknik_accessories/descriptions/brackets/kinova_realsense_camera_adapter/realsense_bracket_for_kinova.dae" /> -->
-    <!--       </geometry> -->
-    <!--     </collision> -->
-    <!--   </link> -->
-    <!--   <joint name="$(arg prefix)wrist_camera_link_visual_joint" type="fixed"> -->
-    <!--     <origin xyz="0 0 0.0" rpy="0 0 0" /> -->
-    <!--     <parent link="$(arg prefix)bracelet_link" /> -->
-    <!--     <child link="$(arg prefix)wrist_camera_link_visual" /> -->
-    <!--   </joint> -->
-    <!-- </xacro:if> -->
     <!-- Visual aids for grasping -->
-    <!-- <link name="finger_tip_closed_point"> -->
-    <!--   <visual> -->
-    <!--     <geometry> -->
-    <!--       <sphere radius="0.007"/> -->
-    <!--     </geometry> -->
-    <!--     <material name=""> -->
-    <!--           <color rgba="0 1.0 0 0.7"/> -->
-    <!--     </material> -->
-    <!--   </visual> -->
-    <!-- </link> -->
-    <!---->
-    <!-- <joint name="finger_tip_closed_point_joint" type="fixed"> -->
-    <!--   <parent link="robotiq_85_base_link"/> -->
-    <!--   <child link = "finger_tip_closed_point"/> -->
-    <!--   <origin xyz="0 0 0.16" rpy="0 0 0"/> -->
-    <!-- </joint> -->
+     <link name="finger_tip_closed_point">
+       <visual>
+         <geometry>
+           <sphere radius="0.007"/>
+         </geometry>
+         <material name="">
+               <color rgba="0 1.0 0 0.7"/>
+         </material>
+       </visual>
+     </link>
+     <joint name="finger_tip_closed_point_joint" type="fixed">
+       <parent link="robotiq_85_base_link"/>
+       <child link = "finger_tip_closed_point"/>
+       <origin xyz="0 0 0.16" rpy="0 0 0"/>
+     </joint>
     <!---->
     <!-- This link aligns the axes of the grasp frame to our required convention for motion planning tasks. -->

Commit message: Align robot description xml

File: src/kinova_gen3_mujoco_config/description/picknik_kinova_gen3.xacro (robot description, xacro)
@@ -523,19 +523,19 @@
     </xacro:cube>
     <!-- Visual aids for grasping -->
-     <link name="finger_tip_closed_point">
-       <visual>
-         <geometry>
-           <sphere radius="0.007"/>
-         </geometry>
-         <material name="">
-               <color rgba="0 1.0 0 0.7"/>
-         </material>
-       </visual>
-     </link>
-     <joint name="finger_tip_closed_point_joint" type="fixed">
-       <parent link="robotiq_85_base_link"/>
-       <child link = "finger_tip_closed_point"/>
-       <origin xyz="0 0 0.16" rpy="0 0 0"/>
-     </joint>
+    <link name="finger_tip_closed_point">
+      <visual>
+        <geometry>
+          <sphere radius="0.007"/>
+        </geometry>
+        <material name="">
+          <color rgba="0 1.0 0 0.7"/>
+        </material>
+      </visual>
+    </link>
+    <joint name="finger_tip_closed_point_joint" type="fixed">
+      <parent link="robotiq_85_base_link"/>
+      <child link = "finger_tip_closed_point"/>
+      <origin xyz="0 0 0.16" rpy="0 0 0"/>
+    </joint>
     <!---->
     <!-- This link aligns the axes of the grasp frame to our required convention for motion planning tasks. -->

Commit message: MuJoCo config fixups
* Change fixed finger joints to continuous joints to get rid of error
  for providing joint states to fixed joints
* Update gripper MuJoCo config to close all the way

Co-authored-by: Paul Gesel <paulgesel@gmail.com>

File: src/kinova_gen3_mujoco_config/description/picknik_kinova_gen3.xacro (robot description, xacro)
@@ -480,12 +480,14 @@
       <mimic joint="robotiq_85_left_knuckle_joint" multiplier="1"/>
     </joint>
-    <joint name="robotiq_85_left_finger_joint" type="fixed">
+    <joint name="robotiq_85_left_finger_joint" type="continuous">
       <parent link="robotiq_85_left_knuckle_link"/>
       <child link="robotiq_85_left_finger_link"/>
+      <axis xyz="0 -1 0"/>
       <origin rpy="0 0 0" xyz="0.03152616 0.0 -0.00376347"/>
     </joint>
-    <joint name="robotiq_85_right_finger_joint" type="fixed">
+    <joint name="robotiq_85_right_finger_joint" type="continuous">
       <parent link="robotiq_85_right_knuckle_link"/>
       <child link="robotiq_85_right_finger_link"/>
+      <axis xyz="0 1 0"/>
       <origin rpy="0 0 0" xyz="-0.03152616 0.0 -0.00376347"/>
     </joint>

Commit message: Add fts_link frame and use in admittance controllers

File: src/kinova_gen3_mujoco_config/description/picknik_kinova_gen3.xacro (robot description, xacro)
@@ -270,4 +270,11 @@
       <axis xyz="0 0 0"/>
     </joint>
+    <link name="fts_link"/>
+    <joint name="fts_joint" type="fixed">
+      <origin rpy="0.0 0.0 3.14159265358979" xyz="0 0 0.0"/>
+      <parent link="end_effector_link"/>
+      <child link="fts_link"/>
+      <axis xyz="0 0 0"/>
+    </joint>
     <!-- Add robotiq 2f 85 gripper model -->
     <link name="robotiq_85_base_link">
@@ -461,7 +468,7 @@
     </link>
     <joint name="robotiq_85_base_joint" type="fixed">
-      <parent link="end_effector_link"/>
+      <parent link="fts_link"/>
       <child link="robotiq_85_base_link"/>
-      <origin rpy="0 0 0" xyz="0 0 0"/>
+      <origin rpy="0 0 -3.14159265358979" xyz="0 0 0"/>
     </joint>
     <joint name="robotiq_85_left_knuckle_joint" type="revolute">

Commit message: Add velocity force controller in MuJoCo config (#35)
* Add VFC test objectives
* Update package.xml dependencies
* Fix FTS site/frame naming & usage

File: src/kinova_gen3_mujoco_config/description/picknik_kinova_gen3.xacro (robot description, xacro)
@@ -271,4 +271,11 @@
       <axis xyz="0 0 0"/>
     </joint>
+    <link name="fts_link"/>
+    <joint name="fts_joint" type="fixed">
+      <origin rpy="0.0 0.0 3.14159265358979" xyz="0 0 0.0"/>
+      <parent link="end_effector_link"/>
+      <child link="fts_link"/>
+      <axis xyz="0 0 0"/>
+    </joint>
     <!-- Add robotiq 2f 85 gripper model -->
     <link name="robotiq_85_base_link">
@@ -462,7 +469,7 @@
     </link>
     <joint name="robotiq_85_base_joint" type="fixed">
-      <parent link="end_effector_link"/>
+      <parent link="fts_link"/>
       <child link="robotiq_85_base_link"/>
-      <origin rpy="0 0 0" xyz="0 0 0"/>
+      <origin rpy="0 0 -3.14159265358979" xyz="0 0 0"/>
     </joint>
     <joint name="robotiq_85_left_knuckle_joint" type="revolute">
